File: ToF_illumination_icHaus_LED.sch (KiCad schematic (older format))
At the start: 41 parts, among them J1 Screw_Terminal_01x02, J2 Conn_01x10, J3 Conn_01x02, J4 Conn_01x02, U1 SN74AUP1T34DCK, U2 MCP1541-TT, U3 iC-HGP, U4 LM2937xT

Commit message: Tantalum capacitors were changed to 1210 size and project was moved to KiCad 5.1.4
Parts:
- C1, C10, C9: footprint Capacitors_Tantalum_SMD:CP_Tantalum_Case-R_EIA-2012-12_Reflow -> Capacitors_SMD:C_1210
Changed lines of the file:
@@
 EESchema Schematic File Version 4
 LIBS:ToF_illumination_icHaus_LED-cache
-EELAYER 29 0
+EELAYER 30 0
 EELAYER END
 $Descr A3 16535 11693
@@
 F 0 "C10" H 5268 5696 50  0000 L CNN
 F 1 "10u" H 5268 5605 50  0000 L CNN
-F 2 "Capacitors_Tantalum_SMD:CP_Tantalum_Case-R_EIA-2012-12_Reflow" H 5188 5500 50  0001 C CNN
+F 2 "Capacitors_SMD:C_1210" H 5188 5500 50  0001 C CNN
 F 3 "~" H 5150 5650 50  0001 C CNN
 	1    5150 5650
@@
 F 0 "C9" H 4568 5696 50  0000 L CNN
 F 1 "100u" H 4568 5605 50  0000 L CNN
-F 2 "Capacitors_Tantalum_SMD:CP_Tantalum_Case-R_EIA-2012-12_Reflow" H 4488 5500 50  0001 C CNN
+F 2 "Capacitors_SMD:C_1210" H 4488 5500 50  0001 C CNN
 F 3 "~" H 4450 5650 50  0001 C CNN
 	1    4450 5650
@@
 F 0 "C1" H 7168 2946 50  0000 L CNN
 F 1 "10u" H 7168 2855 50  0000 L CNN
-F 2 "Capacitors_Tantalum_SMD:CP_Tantalum_Case-R_EIA-2012-12_Reflow" H 7088 2750 50  0001 C CNN
+F 2 "Capacitors_SMD:C_1210" H 7088 2750 50  0001 C CNN
 F 3 "~" H 7050 2900 50  0001 C CNN
 	1    7050 2900

Commit message: Added BOM, improved footprints a bit.
Parts:
- C6, C7, C8: footprint Capacitors_SMD:C_0603 -> Capacitors_SMD:C_0805
- D10, D11, D12: value D_Zener -> uClamp1201H
Changed lines of the file:
@@
 F 0 "C6" H 4735 5154 50  0000 R CNN
 F 1 "1u" H 4735 5245 50  0000 R CNN
-F 2 "Capacitors_SMD:C_0603" H 4888 5050 50  0001 C CNN
+F 2 "Capacitors_SMD:C_0805" H 4888 5050 50  0001 C CNN
 F 3 "~" H 4850 5200 50  0001 C CNN
 	1    4850 5200
@@
 F 0 "C7" H 5185 5154 50  0000 R CNN
 F 1 "1u" H 5185 5245 50  0000 R CNN
-F 2 "Capacitors_SMD:C_0603" H 5338 5050 50  0001 C CNN
+F 2 "Capacitors_SMD:C_0805" H 5338 5050 50  0001 C CNN
 F 3 "~" H 5300 5200 50  0001 C CNN
 	1    5300 5200
@@
 F 0 "C8" H 5635 5154 50  0000 R CNN
 F 1 "1u" H 5635 5245 50  0000 R CNN
-F 2 "Capacitors_SMD:C_0603" H 5788 5050 50  0001 C CNN
+F 2 "Capacitors_SMD:C_0805" H 5788 5050 50  0001 C CNN
 F 3 "~" H 5750 5200 50  0001 C CNN
 	1    5750 5200
@@
 P 5900 2350
 F 0 "D12" H 5900 2566 50  0000 C CNN
-F 1 "D_Zener" H 5900 2475 50  0000 C CNN
+F 1 "uClamp1201H" H 5900 2475 50  0000 C CNN
 F 2 "Diodes_SMD:D_SOD-523" H 5900 2350 50  0001 C CNN
 F 3 "~" H 5900 2350 50  0001 C CNN
@@
 P 5600 1700
 F 0 "D11" H 5600 1916 50  0000 C CNN
-F 1 "D_Zener" H 5600 1825 50  0000 C CNN
+F 1 "uClamp1201H" H 5600 1825 50  0000 C CNN
 F 2 "Diodes_SMD:D_SOD-523" H 5600 1700 50  0001 C CNN
 F 3 "~" H 5600 1700 50  0001 C CNN
@@
 P 5000 1150
 F 0 "D10" H 5000 934 50  0000 C CNN
-F 1 "D_Zener" H 5000 1025 50  0000 C CNN
+F 1 "uClamp1201H" H 5000 1025 50  0000 C CNN
 F 2 "Diodes_SMD:D_SOD-523" H 5000 1150 50  0001 C CNN
 F 3 "~" H 5000 1150 50  0001 C CNN
